File: step_dir_controller_3x2.kicad_pcb (KiCad board)
At the start: 2 copper layers, 69.8 x 40.6 mm, 1 part

Commit message: Changes.
Other:
- board text added: "Janelia Modular Device step_dir_controller part_number: 1241 03/2017 ver 1.0 3x2"
- board text removed: "Janelia Modular Device step_dir_controller part_number: 1000 02/2017 ver 1.0 3x2"
Changed lines of the file:
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@@
-(kicad_pcb (version 20170123) (host pcbnew no-vcs-found-7602~57~ubuntu16.04.1)
+(kicad_pcb (version 20170123) (host pcbnew no-vcs-found-0f0cb64~58~ubuntu16.04.1)
   (general
     (links 0)
     (no_connects 0)
-    (area 0 0 0 0)
+    (area 85.356699 68.211699 155.943301 109.588301)
     (thickness 1.6)
     (drawings 6)
@@
     (effects (font (size 1.016 1.016) (thickness 0.1905)))
   )
-  (gr_text "Janelia Modular Device\nstep_dir_controller\npart_number: 1000\n02/2017 ver 1.0 3x2" (at 89.535 88.9 90) (layer F.SilkS)
+  (gr_text "Janelia Modular Device\nstep_dir_controller\npart_number: 1241\n03/2017 ver 1.0 3x2" (at 89.535 88.9 90) (layer F.SilkS)
     (effects (font (size 1.016 1.016) (thickness 0.254)))
   )

Commit message: Finished v1.0.
Parts:
- added C1: 0.1uF, step_dir_controller_3x2:SM1210, B.Cu at (90.2, 90.2)
- added C2: 0.1uF, step_dir_controller_3x2:SM1210, B.Cu at (120.7, 90.2)
- added C3: 0.1uF, step_dir_controller_3x2:SM1210, B.Cu at (94.6, 80.0)
- added C4: 0.1uF, step_dir_controller_3x2:SM1210, B.Cu at (103.5, 102.2)
- added C5: 0.1uF, step_dir_controller_3x2:SM1210, B.Cu at (115.6, 80.0)
- added C6: 0.1uF, step_dir_controller_3x2:SM1210, B.Cu at (124.5, 102.2)
- added C7: 0.1uF, step_dir_controller_3x2:SM1210, B.Cu at (136.5, 80.0)
- added C8: 0.1uF, step_dir_controller_3x2:SM1210, B.Cu at (145.4, 102.2)
- added CLK1: CLK_32MHZ, step_dir_controller_3x2:CTS_SMD_4_7X5MM, B.Cu at (97.2, 90.2)
- added P1: HEADER_02X05_SMD, step_dir_controller_3x2:HEADER_02x05_SMD, F.Cu at (103.5, 82.5)
- added P2: HEADER_02X05_SMD, step_dir_controller_3x2:HEADER_02x05_SMD, F.Cu at (124.5, 82.5)
- added P3: HEADER_02X05_SMD, step_dir_controller_3x2:HEADER_02x05_SMD, F.Cu at (145.4, 82.5)
- added T1: TERM_BLK_HDR_4POS_VERT_0.138IN, step_dir_controller_3x2:TERM_BLK_HDR_4POS_VERT_0.138IN, F.Cu at (103.5, 98.4)
- added T2: TERM_BLK_HDR_4POS_VERT_0.138IN, step_dir_controller_3x2:TERM_BLK_HDR_4POS_VERT_0.138IN, F.Cu at (124.5, 98.4)
- added T3: TERM_BLK_HDR_4POS_VERT_0.138IN, step_dir_controller_3x2:TERM_BLK_HDR_4POS_VERT_0.138IN, F.Cu at (145.4, 98.4)
- added U1: TMC429, step_dir_controller_3x2:QFN-5x5-32, B.Cu at (113.0, 90.2)
- added U2: 26LS31, step_dir_controller_3x2:SOIC_16_0.154IN, B.Cu at (103.5, 80.0)
- added U3: MAX6817, step_dir_controller_3x2:MAX6817, B.Cu at (103.5, 94.6)
- added U4: 26LS31, step_dir_controller_3x2:SOIC_16_0.154IN, B.Cu at (124.5, 80.0)
- added U5: MAX6817, step_dir_controller_3x2:MAX6817, B.Cu at (124.5, 94.6)
- added U6: 26LS31, step_dir_controller_3x2:SOIC_16_0.154IN, B.Cu at (145.4, 80.0)
- added U7: MAX6817, step_dir_controller_3x2:MAX6817, B.Cu at (145.4, 94.6)
Connections:
- MDB1 pad 10: (no net) -> /CS
- MDB1 pad 11: (no net) -> /MOSI
- MDB1 pad 12: (no net) -> /MISO
- MDB1 pad 13: (no net) -> /SCK
- MDB1 pad 2: (no net) -> /ENABLE_0
- MDB1 pad 3: (no net) -> /ENABLE_1
- MDB1 pad 3V3: (no net) -> +3V3
- MDB1 pad 4: (no net) -> /ENABLE_2
- MDB1 pad 5: (no net) -> /INT
- MDB1 pad 6: (no net) -> /POSCOMP
- MDB1 pad GND: (no net) -> GND
- MDB1 pad VEE: (no net) -> VEE
Routing:
- net GND: track 0.00 -> 310.8 mm
- net +3V3: track 0.00 -> 175.5 mm
- net VEE: track 0.00 -> 94.5 mm, vias 0 -> 1
- net /ENABLE_2: track 0.00 -> 74.9 mm
- net /tmc429_0/DIR_2: track 0.00 -> 48.7 mm
- net /tmc429_0/REF_2: track 0.00 -> 47.5 mm
- net /POSCOMP: track 0.00 -> 39.7 mm, vias 0 -> 1
- net /tmc429_0/REFR_2: track 0.00 -> 36.9 mm, vias 0 -> 2
- net /tmc429_0/STEP_2: track 0.00 -> 36.8 mm
- net /SCK: track 0.00 -> 26.5 mm, vias 0 -> 1
- net /ENABLE_1: track 0.00 -> 23.7 mm, vias 0 -> 1
- net /CS: track 0.00 -> 23.2 mm, vias 0 -> 1
- net /tmc429_0/DIR_0: track 0.00 -> 22.8 mm
- net /MISO: track 0.00 -> 21.2 mm, vias 0 -> 1
- net /tmc429_0/REF_1: track 0.00 -> 20.6 mm
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- added copper zone on B.Cu, net GND
- added copper zone on F.Cu, net GND
Other:
- net class GND: trace_width 0.4064 -> 0.3048
- net class POWER: clearance 0.254 -> 0.1016; trace_width 0.8128 -> 0.3048
- net class SIGNAL: trace_width 0.4064 -> 0.3048
- net class SUPERPOWER: clearance 0.254 -> 0.1016; trace_width 1.2192 -> 0.6096
- board text added: "0"
- board text added: "1"
- board text added: "2"
- board text added: "DIR +"
- board text added: "DIR -"
- board text added: "EN +"
- board text added: "EN -"
- board text added: "GND"
- board text added: "REF"
- board text added: "REFR"
- board text added: "STEP +"
- board text added: "STEP -"
